File: MECHANICAL NUMPAD PCB WITH RP2040/MECHANICAL NUMPAD PCB WITH RP2040.kicad_pcb (KiCad board)
At the start: 4 copper layers, 76.2 x 101.6 mm, 93 parts, among them IC2 RP2040_QFN56, J1 USB_C_Receptacle_USB2.0_16P, SW1 SW_Push, SW10 SW_Push, SW11 SW_Push, SW12 SW_Push, SW13 SW_Push, SW14 SW_Push, SW15 SW_Push, SW16 SW_Push, SW17 SW_Push, SW2 SW_Push, SW21 SKRAAKE010, SW22 SKRAAKE010, SW3 SW_Push, SW4 SW_Push, SW5 SW_Push, SW6 SW_Push, SW7 SW_Push, SW8 SW_Push, SW9 SW_Push, U1 LVL SHFTR, U2 AP2112K-3.3, U5 8MB QSPI Flash, Y1 12MHZ

Commit message: Generating Gerbers and refining PCBs
Parts:
- removed D18, D19, D20, D24, D26, D30: NEOP, LED_SMD:LED_SK6812MINI-E_3.2x2.8mm_P1.5mm_ReverseMount
- added D32: NEOP, LED_SMD:LED_SK6812MINI-E_3.2x2.8mm_P1.5mm_ReverseMount, B.Cu at (57.2, 42.6)
- added D33: NEOP, LED_SMD:LED_SK6812MINI-E_3.2x2.8mm_P1.5mm_ReverseMount, B.Cu at (76.4, 42.6)
- added D35: NEOP, LED_SMD:LED_SK6812MINI-E_3.2x2.8mm_P1.5mm_ReverseMount, B.Cu at (95.4, 42.7)
- added D36: NEOP, LED_SMD:LED_SK6812MINI-E_3.2x2.8mm_P1.5mm_ReverseMount, B.Cu at (57.0, 61.8)
- added D41: NEOP, LED_SMD:LED_SK6812MINI-E_3.2x2.8mm_P1.5mm_ReverseMount, B.Cu at (95.2, 70.8)
- added D42: NEOP, LED_SMD:LED_SK6812MINI-E_3.2x2.8mm_P1.5mm_ReverseMount, F.Cu at (127.3, 60.1)
- added D43: NEOP, LED_SMD:LED_SK6812MINI-E_3.2x2.8mm_P1.5mm_ReverseMount, F.Cu at (127.3, 65.0)
- added D44: NEOP, LED_SMD:LED_SK6812MINI-E_3.2x2.8mm_P1.5mm_ReverseMount, F.Cu at (127.3, 69.9)
- added D45: NEOP, LED_SMD:LED_SK6812MINI-E_3.2x2.8mm_P1.5mm_ReverseMount, F.Cu at (127.3, 74.7)
- added D46: NEOP, LED_SMD:LED_SK6812MINI-E_3.2x2.8mm_P1.5mm_ReverseMount, F.Cu at (127.3, 79.6)
- added D47: NEOP, LED_SMD:LED_SK6812MINI-E_3.2x2.8mm_P1.5mm_ReverseMount, B.Cu at (95.2, 109.1)
- added D48: NEOP, LED_SMD:LED_SK6812MINI-E_3.2x2.8mm_P1.5mm_ReverseMount, B.Cu at (32.8, 26.3)
- added D49: NEOP, LED_SMD:LED_SK6812MINI-E_3.2x2.8mm_P1.5mm_ReverseMount, B.Cu at (38.3, 26.3)
- added D50: NEOP, LED_SMD:LED_SK6812MINI-E_3.2x2.8mm_P1.5mm_ReverseMount, B.Cu at (43.7, 26.3)
- added R13: 200K, Resistor_SMD:R_0603_1608Metric, F.Cu at (141.9, 55.2)
- D31, D40, R13: moved to B.Cu
- D35: renamed from D25; moved to B.Cu
- D37: renamed from D27; moved to B.Cu
- D38: renamed from D28; moved to B.Cu
- D39: renamed from D29; moved to B.Cu
- D42: renamed from D32; moved to B.Cu
- D43: renamed from D33; moved to B.Cu
- D44: renamed from D34; moved to B.Cu
- D45: renamed from D35; moved to B.Cu
- D46: renamed from D36; moved to B.Cu
- U1: footprint Package_SO:VSSOP-8_2.3x2mm_P0.5mm -> Package_DFN_QFN:Texas_S-PVQFN-N14; moved to B.Cu
- moved D42 117.2 mm to (38.1, 99.6)
- moved D45 110.9 mm to (47.7, 118.8)
- moved D46 106.6 mm to (76.2, 118.6)
- moved D31 105.6 mm to (38.0, 42.7)
- moved D38 100.9 mm to (38.1, 80.8)
- moved D43 97.9 mm to (57.4, 99.7)
- moved D35 88.9 mm to (37.9, 61.7)
- moved D39 81.1 mm to (57.3, 80.8)
- moved D44 79.2 mm to (76.3, 100.0)
- moved D40 77.8 mm to (76.2, 80.2)
- moved D37 60.3 mm to (76.4, 61.9)
- moved D38 39.4 mm to (118.8, 74.7)
- moved D37 39.4 mm to (118.8, 69.9)
- moved D39 39.4 mm to (118.8, 79.6)
- moved R13 37.5 mm to (96.5, 50.4), turned to 180 degrees
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Connections:
- D31 pad 2: Net-(D30-DOUT) -> /NEOSIG
- D37 pad 2: Net-(D26-DOUT) -> Net-(D36-DOUT)
- D37 pad 4: Net-(D27-DOUT) -> Net-(D37-DOUT)
- D38 pad 2: Net-(D27-DOUT) -> Net-(D37-DOUT)
- D38 pad 4: Net-(D28-DOUT) -> Net-(D38-DOUT)
- D39 pad 2: Net-(D28-DOUT) -> Net-(D38-DOUT)
- D39 pad 4: Net-(D29-DOUT) -> Net-(D39-DOUT)
- D40 pad 4: unconnected-(D40-DOUT-Pad4) -> Net-(D40-DOUT)
- D42 pad 2: Net-(D31-DOUT) -> Net-(D41-DOUT)
- D46 pad 4: Net-(D36-DOUT) -> Net-(D46-DOUT)
- U1 pad 1: GND -> 3.3V
- U1 pad 2: 3.3V -> /D9
- U1 pad 3: /D9 -> unconnected-(U1-A2-Pad3)
- U1 pad 6: /NEOSIG -> unconnected-(U1-NC-Pad6)
- U1 pad 7: VBUS -> GND
- U1 pad 8: Net-(U1-EN) -> Net-(U1-OE)
Routing:
- net VBUS: track 47.6 -> 523.1 mm, vias 2 -> 36
- net Net-(D47-DOUT): track 0.00 -> 181.5 mm
- net Net-(D41-DOUT): track 0.00 -> 98.4 mm, vias 0 -> 2
- net Net-(D34-DOUT): track 0.00 -> 80.6 mm, vias 0 -> 4
- net /NEOSIG: track 0.00 -> 64.5 mm, vias 0 -> 4
- net Net-(D37-DOUT): track 0.00 -> 60.2 mm, vias 0 -> 2
- net Net-(D44-DOUT): track 0.00 -> 48.1 mm, vias 0 -> 2
- net /D9: track 0.00 -> 38.3 mm, vias 0 -> 2
- net Net-(D45-DOUT): track 0.00 -> 24.6 mm
- net Net-(D46-DOUT): track 0.00 -> 19.8 mm, vias 0 -> 2
- net Net-(D43-DOUT): track 0.00 -> 19.4 mm, vias 0 -> 2
- net Net-(D39-DOUT): track 0.00 -> 18.6 mm, vias 0 -> 4
- net Net-(D31-DOUT): track 0.00 -> 17.4 mm, vias 0 -> 2
- net Net-(D40-DOUT): track 0.00 -> 17.3 mm, vias 0 -> 2
- net Net-(D35-DOUT): track 0.00 -> 16.9 mm, vias 0 -> 2
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- added copper zone on In1.Cu, net GND
- removed copper zone on In1.Cu, net 3.3V
Other:
- board text added: "ICARUS RESEARCH INSTITUTE"
