File: 2 LAYER MECHANICAL NUMPAD PCB WITH RP2040/2 LAYER MECHANICAL NUMPAD PCB WITH RP2040.kicad_sch (KiCad schematic)
At the start: 93 parts, among them IC2 RP2040_QFN56, J1 USB_C_Receptacle_USB2.0_16P, SW1 SW_Push, SW10 SW_Push, SW11 SW_Push, SW12 SW_Push, SW13 SW_Push, SW14 SW_Push, SW15 SW_Push, SW16 SW_Push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

Commit message: Created files
Parts:
- D31, D32, D33, D34, D35, D36, D37, D38, D39, D40, D41, D42, D43, D44, D45, D46, D47, D48, D49, D50: footprint LED_SMD:LED_SK6812MINI-E_3.2x2.8mm_P1.5mm_ReverseMount -> JH_FOOTPRINTS:LED_SK6812MINI-E_3.2x2.8mm_P1.5mm_ReverseMount
Changed lines of the file:
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@@
 			)
 		)
-		(property "Footprint" "LED_SMD:LED_SK6812MINI-E_3.2x2.8mm_P1.5mm_ReverseMount"
+		(property "Footprint" "JH_FOOTPRINTS:LED_SK6812MINI-E_3.2x2.8mm_P1.5mm_ReverseMount"
 			(at 92.71 219.71 0)
 			(hide yes)
@@
 			)
 		)
-		(property "Footprint" "LED_SMD:LED_SK6812MINI-E_3.2x2.8mm_P1.5mm_ReverseMount"
+		(property "Footprint" "JH_FOOTPRINTS:LED_SK6812MINI-E_3.2x2.8mm_P1.5mm_ReverseMount"
 			(at 31.75 262.89 0)
 			(hide yes)
@@
 			)
 		)
-		(property "Footprint" "LED_SMD:LED_SK6812MINI-E_3.2x2.8mm_P1.5mm_ReverseMount"
+		(property "Footprint" "JH_FOOTPRINTS:LED_SK6812MINI-E_3.2x2.8mm_P1.5mm_ReverseMount"
 			(at 62.23 241.3 0)
 			(hide yes)
@@
 			)
 		)
-		(property "Footprint" "LED_SMD:LED_SK6812MINI-E_3.2x2.8mm_P1.5mm_ReverseMount"
+		(property "Footprint" "JH_FOOTPRINTS:LED_SK6812MINI-E_3.2x2.8mm_P1.5mm_ReverseMount"
 			(at 62.23 219.71 0)
 			(hide yes)
@@
 			)
 		)
-		(property "Footprint" "LED_SMD:LED_SK6812MINI-E_3.2x2.8mm_P1.5mm_ReverseMount"
+		(property "Footprint" "JH_FOOTPRINTS:LED_SK6812MINI-E_3.2x2.8mm_P1.5mm_ReverseMount"
 			(at 77.47 241.3 0)
 			(hide yes)
@@
 			)
 		)
-		(property "Footprint" "LED_SMD:LED_SK6812MINI-E_3.2x2.8mm_P1.5mm_ReverseMount"
+		(property "Footprint" "JH_FOOTPRINTS:LED_SK6812MINI-E_3.2x2.8mm_P1.5mm_ReverseMount"
 			(at 31.75 219.71 0)
 			(hide yes)
@@
 			)
 		)
-		(property "Footprint" "LED_SMD:LED_SK6812MINI-E_3.2x2.8mm_P1.5mm_ReverseMount"
+		(property "Footprint" "JH_FOOTPRINTS:LED_SK6812MINI-E_3.2x2.8mm_P1.5mm_ReverseMount"
 			(at 62.23 262.89 0)
 			(hide yes)
@@
 			)
 		)
-		(property "Footprint" "LED_SMD:LED_SK6812MINI-E_3.2x2.8mm_P1.5mm_ReverseMount"
+		(property "Footprint" "JH_FOOTPRINTS:LED_SK6812MINI-E_3.2x2.8mm_P1.5mm_ReverseMount"
 			(at 92.71 284.48 0)
 			(hide yes)
@@
 			)
 		)
-		(property "Footprint" "LED_SMD:LED_SK6812MINI-E_3.2x2.8mm_P1.5mm_ReverseMount"
+		(property "Footprint" "JH_FOOTPRINTS:LED_SK6812MINI-E_3.2x2.8mm_P1.5mm_ReverseMount"
 			(at 92.71 262.89 0)
 			(hide yes)
@@
 			)
 		)
-		(property "Footprint" "LED_SMD:LED_SK6812MINI-E_3.2x2.8mm_P1.5mm_ReverseMount"
+		(property "Footprint" "JH_FOOTPRINTS:LED_SK6812MINI-E_3.2x2.8mm_P1.5mm_ReverseMount"
 			(at 46.99 262.89 0)
 			(hide yes)
@@
 			)
 		)
-		(property "Footprint" "LED_SMD:LED_SK6812MINI-E_3.2x2.8mm_P1.5mm_ReverseMount"
+		(property "Footprint" "JH_FOOTPRINTS:LED_SK6812MINI-E_3.2x2.8mm_P1.5mm_ReverseMount"
 			(at 77.47 284.48 0)
 			(hide yes)
@@
 			)
 		)
-		(property "Footprint" "LED_SMD:LED_SK6812MINI-E_3.2x2.8mm_P1.5mm_ReverseMount"
+		(property "Footprint" "JH_FOOTPRINTS:LED_SK6812MINI-E_3.2x2.8mm_P1.5mm_ReverseMount"
 			(at 77.47 262.89 0)
 			(hide yes)
@@
 			)
 		)
-		(property "Footprint" "LED_SMD:LED_SK6812MINI-E_3.2x2.8mm_P1.5mm_ReverseMount"
+		(property "Footprint" "JH_FOOTPRINTS:LED_SK6812MINI-E_3.2x2.8mm_P1.5mm_ReverseMount"
 			(at 46.99 241.3 0)
 			(hide yes)
@@
 			)
 		)
-		(property "Footprint" "LED_SMD:LED_SK6812MINI-E_3.2x2.8mm_P1.5mm_ReverseMount"
+		(property "Footprint" "JH_FOOTPRINTS:LED_SK6812MINI-E_3.2x2.8mm_P1.5mm_ReverseMount"
 			(at 92.71 241.3 0)
 			(hide yes)
@@
 			)
 		)
-		(property "Footprint" "LED_SMD:LED_SK6812MINI-E_3.2x2.8mm_P1.5mm_ReverseMount"
+		(property "Footprint" "JH_FOOTPRINTS:LED_SK6812MINI-E_3.2x2.8mm_P1.5mm_ReverseMount"
 			(at 31.75 284.48 0)
 			(hide yes)
@@
 			)
 		)
-		(property "Footprint" "LED_SMD:LED_SK6812MINI-E_3.2x2.8mm_P1.5mm_ReverseMount"
+		(property "Footprint" "JH_FOOTPRINTS:LED_SK6812MINI-E_3.2x2.8mm_P1.5mm_ReverseMount"
 			(at 77.47 219.71 0)
 			(hide yes)
@@
 			)
 		)
-		(property "Footprint" "LED_SMD:LED_SK6812MINI-E_3.2x2.8mm_P1.5mm_ReverseMount"
+		(property "Footprint" "JH_FOOTPRINTS:LED_SK6812MINI-E_3.2x2.8mm_P1.5mm_ReverseMount"
 			(at 31.75 241.3 0)
 			(hide yes)
@@
 			)
 		)
-		(property "Footprint" "LED_SMD:LED_SK6812MINI-E_3.2x2.8mm_P1.5mm_ReverseMount"
+		(property "Footprint" "JH_FOOTPRINTS:LED_SK6812MINI-E_3.2x2.8mm_P1.5mm_ReverseMount"
 			(at 46.99 219.71 0)
 			(hide yes)
@@
 			)
 		)
-		(property "Footprint" "LED_SMD:LED_SK6812MINI-E_3.2x2.8mm_P1.5mm_ReverseMount"
+		(property "Footprint" "JH_FOOTPRINTS:LED_SK6812MINI-E_3.2x2.8mm_P1.5mm_ReverseMount"
 			(at 46.99 284.48 0)
 			(hide yes)
@@
 			)
 		)
-		(property "Footprint" "LED_SMD:LED_SK6812MINI-E_3.2x2.8mm_P1.5mm_ReverseMount"
+		(property "Footprint" "JH_FOOTPRINTS:LED_SK6812MINI-E_3.2x2.8mm_P1.5mm_ReverseMount"
 			(at 62.23 284.48 0)
 			(hide yes)
